Commit message: Fix the xacro file that cause ros2_control of gripper inactivated

File: robotiq_description/urdf/2f_140.ros2_control.xacro (robot description, xacro)
@@ -10,10 +10,5 @@
         use_fake_hardware:=false
         mock_sensor_commands:=false
-        com_port:=/dev/ttyUSB0
-        gripper_speed_multiplier:=1.0
-        gripper_force_multiplier:=0.5
-        gripper_max_speed:=0.250
-        gripper_max_force:=125.0
-        gripper_closed_position:=0.695">
+        com_port:=/dev/ttyUSB0">
         <ros2_control name="${name}" type="system">
             <!-- Plugins -->
@@ -24,6 +19,9 @@
                     <param name="joint_states_topic">${isaac_joint_states}</param>
                 </xacro:if>
+                <!-- <xacro:if value="${sim_gazebo}">
+                    <plugin>ign_ros2_control/IgnitionSystem</plugin>
+                </xacro:if> -->
                 <xacro:if value="${sim_gazebo}">
-                    <plugin>ign_ros2_control/IgnitionSystem</plugin>
+                    <plugin>gazebo_ros2_control/GazeboSystem</plugin>
                 </xacro:if>
                 <xacro:if value="${use_fake_hardware}">
@@ -34,10 +32,8 @@
                 <xacro:unless value="${use_fake_hardware or sim_gazebo or sim_isaac}">
                     <plugin>robotiq_driver/RobotiqGripperHardwareInterface</plugin>
-                    <param name="gripper_closed_position">${gripper_closed_position}</param>
+                    <param name="gripper_closed_position">0.695</param>
                     <param name="COM_port">${com_port}</param>
-                    <param name="gripper_speed_multiplier">${gripper_speed_multiplier}</param>
-                    <param name="gripper_force_multiplier">${gripper_force_multiplier}</param>
-                    <param name="gripper_max_speed">${gripper_max_speed}</param>
-                    <param name="gripper_max_force">${gripper_max_force}</param>
+                    <param name="gripper_speed_multiplier">1.0</param>
+                    <param name="gripper_force_multiplier">0.5</param>
                 </xacro:unless>
             </hardware>
@@ -47,5 +43,5 @@
                 <command_interface name="position" />
                 <state_interface name="position">
-                    <param name="initial_value">${gripper_closed_position}</param>
+                    <param name="initial_value">0.695</param>
                 </state_interface>
                 <state_interface name="velocity"/>
@@ -54,4 +50,6 @@
             <xacro:if value="${use_fake_hardware or sim_isaac or sim_gazebo}">
                 <joint name="${prefix}left_inner_knuckle_joint">
+                    <param name="mimic">${prefix}finger_joint</param>
+                    <param name="multiplier">-1</param>
                     <xacro:unless value="${sim_gazebo}">
                         <state_interface name="position"/>
@@ -60,4 +58,6 @@
                 </joint>
                 <joint name="${prefix}left_inner_finger_joint">
+                    <param name="mimic">${prefix}finger_joint</param>
+                    <param name="multiplier">1</param>
                     <xacro:unless value="${sim_gazebo}">
                         <state_interface name="position"/>
@@ -66,4 +66,6 @@
                 </joint>
                 <joint name="${prefix}right_outer_knuckle_joint">
+                    <param name="mimic">${prefix}finger_joint</param>
+                    <param name="multiplier">-1</param>
                     <xacro:unless value="${sim_gazebo}">
                         <state_interface name="position"/>
@@ -72,4 +74,6 @@
                 </joint>
                 <joint name="${prefix}right_inner_knuckle_joint">
+                    <param name="mimic">${prefix}finger_joint</param>
+                    <param name="multiplier">-1</param>
                     <xacro:unless value="${sim_gazebo}">
                         <state_interface name="position"/>
@@ -78,4 +82,6 @@
                 </joint>
                 <joint name="${prefix}right_inner_finger_joint">
+                    <param name="mimic">${prefix}finger_joint</param>
+                    <param name="multiplier">1</param>
                     <xacro:unless value="${sim_gazebo}">
                         <state_interface name="position"/>

File: robotiq_description/urdf/2f_85.ros2_control.xacro (robot description, xacro)
@@ -10,10 +10,5 @@
         use_fake_hardware:=false
         mock_sensor_commands:=false
-        com_port:=/dev/ttyUSB0
-        gripper_speed_multiplier:=1.0
-        gripper_force_multiplier:=0.5
-        gripper_max_speed:=0.150
-        gripper_max_force:=235.0
-        gripper_closed_position:=0.7929">
+        com_port:=/dev/ttyUSB0">
         <ros2_control name="${name}" type="system">
             <!-- Plugins -->
@@ -27,6 +22,9 @@
                     <param name="trigger_joint_command_threshold">0.02</param>
                 </xacro:if>
+                <!-- <xacro:if value="${sim_gazebo}">
+                    <plugin>ign_ros2_control/IgnitionSystem</plugin>
+                </xacro:if> -->
                 <xacro:if value="${sim_gazebo}">
-                    <plugin>ign_ros2_control/IgnitionSystem</plugin>
+                    <plugin>gazebo_ros2_control/GazeboSystem</plugin>
                 </xacro:if>
                 <xacro:if value="${use_fake_hardware}">
@@ -37,10 +35,8 @@
                 <xacro:unless value="${use_fake_hardware or sim_gazebo or sim_isaac}">
                     <plugin>robotiq_driver/RobotiqGripperHardwareInterface</plugin>
-                    <param name="gripper_closed_position">${gripper_closed_position}</param>
+                    <param name="gripper_closed_position">0.7929</param>
                     <param name="COM_port">${com_port}</param>
-                    <param name="gripper_speed_multiplier">${gripper_speed_multiplier}</param>
-                    <param name="gripper_force_multiplier">${gripper_force_multiplier}</param>
-                    <param name="gripper_max_speed">${gripper_max_speed}</param>
-                    <param name="gripper_max_force">${gripper_max_force}</param>
+                    <param name="gripper_speed_multiplier">1.0</param>
+                    <param name="gripper_force_multiplier">0.5</param>
                 </xacro:unless>
             </hardware>
@@ -50,5 +46,5 @@
                 <command_interface name="position" />
                 <state_interface name="position">
-                    <param name="initial_value">${gripper_closed_position}</param>
+                    <param name="initial_value">0.7929</param>
                 </state_interface>
                 <state_interface name="velocity"/>
@@ -57,4 +53,6 @@
             <xacro:if value="${use_fake_hardware or sim_isaac or sim_gazebo}">
                 <joint name="${prefix}robotiq_85_right_knuckle_joint">
+                    <param name="mimic">${prefix}robotiq_85_left_knuckle_joint</param>
+                    <param name="multiplier">-1</param>
                     <xacro:unless value="${sim_gazebo}">
                         <state_interface name="position"/>
@@ -63,4 +61,6 @@
                 </joint>
                 <joint name="${prefix}robotiq_85_left_inner_knuckle_joint">
+                    <param name="mimic">${prefix}robotiq_85_left_knuckle_joint</param>
+                    <param name="multiplier">1</param>
                     <xacro:unless value="${sim_gazebo}">
                         <state_interface name="position"/>
@@ -69,4 +69,6 @@
                 </joint>
                 <joint name="${prefix}robotiq_85_right_inner_knuckle_joint">
+                    <param name="mimic">${prefix}robotiq_85_left_knuckle_joint</param>
+                    <param name="multiplier">-1</param>
                     <xacro:unless value="${sim_gazebo}">
                         <state_interface name="position"/>
@@ -75,4 +77,6 @@
                 </joint>
                 <joint name="${prefix}robotiq_85_left_finger_tip_joint">
+                    <param name="mimic">${prefix}robotiq_85_left_knuckle_joint</param>
+                    <param name="multiplier">-1</param>
                     <xacro:unless value="${sim_gazebo}">
                         <state_interface name="position"/>
@@ -81,4 +85,6 @@
                 </joint>
                 <joint name="${prefix}robotiq_85_right_finger_tip_joint">
+                    <param name="mimic">${prefix}robotiq_85_left_knuckle_joint</param>
+                    <param name="multiplier">1</param>
                     <xacro:unless value="${sim_gazebo}">
                         <state_interface name="position"/>

File: robotiq_description/urdf/robotiq_2f_140.xacro (robot description, xacro)
@@ -161,5 +161,5 @@
       <axis xyz="1 0 0" />
       <limit lower="-0.725" upper="0.725" velocity="2.0" effort="1000" />
-    <mimic joint="${prefix}finger_joint" multiplier="-1" offset="0" />
+      <mimic joint="${prefix}finger_joint" multiplier="-1" offset="0" />
     </joint>
     <xacro:finger_joints prefix="${prefix}" fingerprefix="right" reflect="-1.0"/>

File: robotiq_description/urdf/robotiq_2f_85_macro.urdf.xacro (robot description, xacro)
@@ -13,10 +13,5 @@
         mock_sensor_commands:=false
         include_ros2_control:=true
-        com_port:=/dev/ttyUSB0
-        gripper_speed_multiplier:=1.0
-        gripper_force_multiplier:=0.5
-        gripper_max_speed:=0.150
-        gripper_max_force:=235.0
-        gripper_closed_position:=0.7929">
+        com_port:=/dev/ttyUSB0">
         <!-- ros2 control include -->
         <xacro:include filename="$(find robotiq_description)/urdf/2f_85.ros2_control.xacro" />
@@ -31,10 +26,5 @@
                 use_fake_hardware="${use_fake_hardware}"
                 mock_sensor_commands="${mock_sensor_commands}"
-                com_port="${com_port}"
-                gripper_speed_multiplier="${gripper_speed_multiplier}"
-                gripper_force_multiplier="${gripper_force_multiplier}"
-                gripper_max_speed="${gripper_max_speed}"
-                gripper_max_force="${gripper_max_force}"
-                gripper_closed_position="${gripper_closed_position}"/>
+                com_port="${com_port}"/>
         </xacro:if>
         <link name="${prefix}robotiq_85_base_link">
@@ -237,5 +227,5 @@
             <axis xyz="0 -1 0" />
             <origin xyz="0.03060114 0.0 0.05490452" rpy="0 0 0" />
-            <limit lower="0.0" upper="0.8" velocity="0.5" effort="50" />
+            <limit lower="0.0" upper="0.8" velocity="0.5" effort="5" />
         </joint>
         <joint name="${prefix}robotiq_85_right_knuckle_joint" type="revolute">
@@ -244,5 +234,5 @@
             <axis xyz="0 -1 0" />
             <origin xyz="-0.03060114 0.0 0.05490452" rpy="0 0 0" />
-            <limit lower="-0.8" upper="0.0" velocity="0.5" effort="50" />
+            <limit lower="-0.8" upper="0.0" velocity="0.5" effort="5" />
             <mimic joint="${prefix}robotiq_85_left_knuckle_joint" multiplier="-1" />
         </joint>
